Commit message: Fix cameras urdf

File: urdf/cameras.urdf.xacro (robot description, xacro)
@@ -10,5 +10,5 @@
    <link name="camera5_link"/>
    <joint name="joint_lidar_camera0" type="fixed">
-    <parent link="lslidarc16" />
+    <parent link="velodyne" />
     <child link="camera0_link" />
     <!--origin xyz="0.15809 0.12394 -0.08268" rpy="-1.167301 0.102245 0.949740" /--> <!--Before origin changed-->
@@ -16,5 +16,5 @@
    </joint>
    <joint name="joint_lidar_camera1" type="fixed">
-    <parent link="lslidarc16" />
+    <parent link="velodyne" />
     <child link="camera1_link" />
     <!--origin xyz="0.34382 0.09629 -0.08268" rpy="-1.3634311444 0.165909317 -0.318686332" /--> <!--Before origin changed-->
@@ -22,5 +22,5 @@
    </joint>
    <joint name="joint_lidar_camera2" type="fixed">
-    <parent link="lslidarc16" />
+    <parent link="velodyne" />
     <child link="camera2_link" />
     <!--origin xyz="0.41006 -0.03625 -0.08268" rpy="-1.48352986 0 -1.57079632" /--> <!--Before origin changed-->
@@ -28,5 +28,5 @@
    </joint>
    <joint name="joint_lidar_camera3" type="fixed">
-    <parent link="lslidarc16" />
+    <parent link="velodyne" />
     <child link="camera3_link" />
     <!--origin xyz="0.27487 -0.11869 -0.08268" rpy="-1.3634311444 -0.165909317 -2.82290632" /--> <!--Before origin changed-->
@@ -34,5 +34,5 @@
    </joint>
    <joint name="joint_lidar_camera4" type="fixed">
-    <parent link="lslidarc16" />
+    <parent link="velodyne" />
     <child link="camera4_link" />
     <!--origin xyz="0.11548 -0.06528 -0.08268" rpy="-1.167301 -0.102245 2.19185" /--> <!--Before origin changed-->
@@ -40,5 +40,5 @@
    </joint>
    <joint name="joint_lidar_camera5" type="fixed">
-    <parent link="lslidarc16" />
+    <parent link="velodyne" />
     <child link="camera5_link" />
     <!--origin xyz="0.33903 0 0.05769" rpy="0.1745329 0 1.57079632" /--> <!--Before origin changed-->

Commit message: Temporally commit to save old configuration

File: urdf/cameras.urdf.xacro (robot description, xacro)
@@ -3,7 +3,13 @@
    <xacro:property name="M_PI" value="3.1415926535897931"/>
    <xacro:property name="length_cam" value="0.05" />
-   <link name="camera0_link"/>
+   <link name="camera2_link"/>
+   <joint name="joint_lidar_camera2" type="fixed">
+    <parent link="lslidarc16" />
+    <child link="camera2_link" />
+    <!--origin xyz="0.41006 -0.03625 -0.08268" rpy="-1.48352986 0 -1.57079632" /--> <!--Before origin changed-->
+    <origin xyz="0.45576 -0.03625 -0.07258" rpy="-1.48352986 0 -1.57079632" /> <!--After origin changed-->
+   </joint>
+   <!--link name="camera0_link"/>
    <link name="camera1_link"/>
-   <link name="camera2_link"/>
    <link name="camera3_link"/>
    <link name="camera4_link"/>
@@ -12,36 +18,25 @@
     <parent link="lslidarc16" />
     <child link="camera0_link" />
-    <!--origin xyz="0.15809 0.12394 -0.08268" rpy="-1.167301 0.102245 0.949740" /--> <!--Before origin changed-->
-    <origin xyz="0.12759 0.1461 -0.07258" rpy="-1.167301 0.102245 0.949740" /> <!-- After origin changed-->
+    <origin xyz="0.12759 0.1461 -0.07258" rpy="-1.167301 0.102245 0.949740" />
    </joint>
    <joint name="joint_lidar_camera1" type="fixed">
     <parent link="lslidarc16" />
     <child link="camera1_link" />
-    <!--origin xyz="0.34382 0.09629 -0.08268" rpy="-1.3634311444 0.165909317 -0.318686332" /--> <!--Before origin changed-->
-    <origin xyz="0.35547 0.13215 -0.07258" rpy="-1.3634311444 0.165909317 -0.318686332" /> <!--After origin changed-->
-   </joint>
-   <joint name="joint_lidar_camera2" type="fixed">
-    <parent link="lslidarc16" />
-    <child link="camera2_link" />
-    <!--origin xyz="0.41006 -0.03625 -0.08268" rpy="-1.48352986 0 -1.57079632" /--> <!--Before origin changed-->
-    <origin xyz="0.45576 -0.03625 -0.07258" rpy="-1.48352986 0 -1.57079632" /> <!--After origin changed-->
+    <origin xyz="0.35547 0.13215 -0.07258" rpy="-1.3634311444 0.165909317 -0.318686332" />
    </joint>
    <joint name="joint_lidar_camera3" type="fixed">
     <parent link="lslidarc16" />
     <child link="camera3_link" />
-    <!--origin xyz="0.27487 -0.11869 -0.08268" rpy="-1.3634311444 -0.165909317 -2.82290632" /--> <!--Before origin changed-->
-    <origin xyz="0.28652 -0.15455 -0.07258" rpy="-1.3634311444 -0.165909317 -2.82290632" /> <!--After origin changed-->
+    <origin xyz="0.28652 -0.15455 -0.07258" rpy="-1.3634311444 -0.165909317 -2.82290632" />
    </joint>
    <joint name="joint_lidar_camera4" type="fixed">
     <parent link="lslidarc16" />
     <child link="camera4_link" />
-    <!--origin xyz="0.11548 -0.06528 -0.08268" rpy="-1.167301 -0.102245 2.19185" /--> <!--Before origin changed-->
-    <origin xyz="0.08497 -0.08744 -0.07258" rpy="-1.167301 -0.102245 2.19185" /> <!--After origin changed-->
+    <origin xyz="0.08497 -0.08744 -0.07258" rpy="-1.167301 -0.102245 2.19185" />
    </joint>
    <joint name="joint_lidar_camera5" type="fixed">
     <parent link="lslidarc16" />
     <child link="camera5_link" />
-    <!--origin xyz="0.33903 0 0.05769" rpy="0.1745329 0 1.57079632" /--> <!--Before origin changed-->
-    <origin xyz="0.33403 0 0.11308" rpy="0.1745329 0 1.57079632" /> <!--After origin changed-->
-   </joint>
+    <origin xyz="0.33403 0 0.11308" rpy="0.1745329 0 1.57079632" />
+   </joint-->
 </robot>

File: urdf/marmotte.urdf.xacro (robot description, xacro)
@@ -9,10 +9,10 @@
     <child link="lslidarc16" />
   </joint>
-  <link name="realsense_link"/>
+  <!--link name="realsense_link"/>
   <joint name="realsense_joint" type="fixed">
     <origin xyz="-0.31593 -0.0175 0.34488" rpy="0 0.558505 ${M_PI}" />
     <parent link="base_link" />
     <child link="realsense_link" />
-  </joint>
+  </joint-->
   <!-- Cameras -->
   <xacro:include filename="$(find marmotte_description)/urdf/cameras.urdf.xacro"/>
