Commit message: Added changed to tf static

File: urdf/marmotte.urdf.xacro (robot description, xacro)
@@ -1,11 +1,19 @@
 <?xml version="1.0"?>
-<robot name="husky" xmlns:xacro="http://ros.org/wiki/xacro">
+<robot name="marmotte" xmlns:xacro="http://ros.org/wiki/xacro">
   <xacro:property name="M_PI" value="3.14159"/>
   <link name="base_link"/>
   <link name="lslidarc16"/>
   <joint name="lslidarc16_joint" type="fixed">
-    <origin xyz="0.31934 0 0.25611" rpy="0 -0.174533 ${M_PI}" />
+    <origin xyz="0.25834 0 0.30611" rpy="0 -0.178 ${M_PI}" />
     <parent link="base_link" />
     <child link="lslidarc16" />
   </joint>
+  <link name="realsense_link"/>
+  <joint name="realsense_joint" type="fixed">
+    <origin xyz="-0.31593 -0.0175 0.34488" rpy="0 0.558505 ${M_PI}" />
+    <parent link="base_link" />
+    <child link="realsense_link" />
+  </joint>
+  <!-- Cameras -->
+  <xacro:include filename="$(find marmotte_description)/urdf/cameras.urdf.xacro"/>
 </robot>

Commit message: Add tfs for new shared lidar-imu panel

File: urdf/marmotte.urdf.xacro (robot description, xacro)
@@ -3,9 +3,40 @@
   <xacro:property name="M_PI" value="3.14159"/>
   <link name="base_link"/>
+  <link name="lidar_imu_mount_horizontal"/>
+  <joint name="lidar_imu_mount_horizontal_joint" type="fixed">
+      <origin xyz="0.19834 0.06 0.26011" rpy="0 -0.178 0" />
+      <parent link="base_link" />
+      <child link="lidar_imu_mount_horizontal" />
+  </joint>
+  <link name="lidar_imu_board"/>
+  <joint name="lidar_imu_board_joint" type="fixed">
+      <origin xyz="0 0 0.039" rpy="0 0 0" />
+      <parent link="lidar_imu_mount_horizontal" />
+      <child link="lidar_imu_board" />
+  </joint>
+  <!-- Vertical board -->
+  <!-- <link name="lidar_imu_mount_vertical"/>
+  <joint name="lidar_imu_mount_vertical_joint" type="fixed">
+      <origin xyz="0 0 0" rpy="0 0.0 ${M_PI}" />
+      <parent link="base_link" />
+      <child link="lidar_imu_mount_vertical" />
+  </joint> -->
+    <!-- <link name="lidar_imu_board"/>
+    <joint name="lidar_imu_board_joint" type="fixed">
+        <origin xyz="0.25834 0 0.30611" rpy="0 -0.178 ${M_PI}" />
+        <parent link="lidar_imu_mount_vertical" />
+        <child link="lidar_imu_board" />
+    </joint> -->
   <link name="lslidarc16"/>
   <joint name="lslidarc16_joint" type="fixed">
-    <origin xyz="0.25834 0 0.30611" rpy="0 -0.178 ${M_PI}" />
-    <parent link="base_link" />
+    <origin xyz="0.06 -0.06 0.036" rpy="0 0 ${M_PI/2}" />
+    <parent link="lidar_imu_board" />
     <child link="lslidarc16" />
+  </joint>
+  <link name="imu"/>
+  <joint name="imu_joint" type="fixed">
+    <origin xyz="0.039254 -0.04274357 -0.0161" rpy="$(M_PI) 0 0" />
+    <parent link="lidar_imu_board" />
+    <child link="imu" />
   </joint>
   <link name="realsense_link"/>

Commit message: Fix M_PI

File: urdf/marmotte.urdf.xacro (robot description, xacro)
@@ -30,5 +30,5 @@
   <link name="lslidarc16"/>
   <joint name="lslidarc16_joint" type="fixed">
-    <origin xyz="0.06 -0.06 0.036" rpy="0 0 ${M_PI/2}" />
+    <origin xyz="0.06 -0.06 0.036" rpy="0 0 ${M_PI}/2" />
     <parent link="lidar_imu_board" />
     <child link="lslidarc16" />
@@ -36,5 +36,5 @@
   <link name="imu"/>
   <joint name="imu_joint" type="fixed">
-    <origin xyz="0.039254 -0.04274357 -0.0161" rpy="$(M_PI) 0 0" />
+    <origin xyz="0.039254 -0.04274357 -0.0161" rpy="${M_PI} 0 0" />
     <parent link="lidar_imu_board" />
     <child link="imu" />

Commit message: Fix M_PI

File: urdf/marmotte.urdf.xacro (robot description, xacro)
@@ -30,5 +30,5 @@
   <link name="lslidarc16"/>
   <joint name="lslidarc16_joint" type="fixed">
-    <origin xyz="0.06 -0.06 0.036" rpy="0 0 ${M_PI}/2" />
+    <origin xyz="0.06 -0.06 0.036" rpy="0 0 ${M_PI/2}" />
     <parent link="lidar_imu_board" />
     <child link="lslidarc16" />

Commit message: Add other calibration configurations

File: urdf/marmotte.urdf.xacro (robot description, xacro)
@@ -2,30 +2,40 @@
 <robot name="marmotte" xmlns:xacro="http://ros.org/wiki/xacro">
   <xacro:property name="M_PI" value="3.14159"/>
+  <!-- horizontal, horizontal_90, vertical -->
+  <xacro:property name="configuration" value="horizontal"/>
   <link name="base_link"/>
-  <link name="lidar_imu_mount_horizontal"/>
-  <joint name="lidar_imu_mount_horizontal_joint" type="fixed">
-      <origin xyz="0.19834 0.06 0.26011" rpy="0 -0.178 0" />
-      <parent link="base_link" />
-      <child link="lidar_imu_mount_horizontal" />
-  </joint>
+  <xacro:if value="${configuration != 'vertical'}">
+    <link name="lidar_imu_mount_horizontal"/>
+    <joint name="lidar_imu_mount_horizontal_joint" type="fixed">
+        <origin xyz="0.19834 0.06 0.26011" rpy="0 0.178 0" />
+        <parent link="base_link" />
+        <child link="lidar_imu_mount_horizontal" />
+    </joint>
+  </xacro:if>
+  <!-- Vertical board -->
+  <xacro:if value="${configuration == 'vertical'}">
+    <link name="lidar_imu_mount_vertical"/>
+    <joint name="lidar_imu_mount_vertical_joint" type="fixed">
+        <origin xyz="0.17834 -0.02 0.38378" rpy="${M_PI/2} 0.178 0" />
+        <parent link="base_link" />
+        <child link="lidar_imu_mount_vertical" />
+    </joint>
+  </xacro:if>
   <link name="lidar_imu_board"/>
   <joint name="lidar_imu_board_joint" type="fixed">
-      <origin xyz="0 0 0.039" rpy="0 0 0" />
-      <parent link="lidar_imu_mount_horizontal" />
+      <xacro:if value="${configuration != 'horizontal_90'}">
+        <origin xyz="0 0 0.039" rpy="0 0 0" />
+      </xacro:if>
+      <xacro:if value="${configuration == 'horizontal_90'}">
+        <origin xyz="0 0 0.039" rpy="0 0 ${M_PI/2}" />
+      </xacro:if>
+      <xacro:if value="${configuration != 'vertical'}">
+        <parent link="lidar_imu_mount_horizontal" />
+      </xacro:if>
+      <xacro:if value="${configuration == 'vertical'}">
+        <parent link="lidar_imu_mount_vertical" />
+      </xacro:if>
       <child link="lidar_imu_board" />
   </joint>
-  <!-- Vertical board -->
-  <!-- <link name="lidar_imu_mount_vertical"/>
-  <joint name="lidar_imu_mount_vertical_joint" type="fixed">
-      <origin xyz="0 0 0" rpy="0 0.0 ${M_PI}" />
-      <parent link="base_link" />
-      <child link="lidar_imu_mount_vertical" />
-  </joint> -->
-    <!-- <link name="lidar_imu_board"/>
-    <joint name="lidar_imu_board_joint" type="fixed">
-        <origin xyz="0.25834 0 0.30611" rpy="0 -0.178 ${M_PI}" />
-        <parent link="lidar_imu_mount_vertical" />
-        <child link="lidar_imu_board" />
-    </joint> -->
   <link name="lslidarc16"/>
   <joint name="lslidarc16_joint" type="fixed">
@@ -47,4 +57,4 @@
   </joint>
   <!-- Cameras -->
-  <xacro:include filename="$(find marmotte_description)/urdf/cameras.urdf.xacro"/>
+  <!-- <xacro:include filename="$(find marmotte_description)/urdf/cameras.urdf.xacro"/> -->
 </robot>

Commit message: Move lidar_imu_board origin from the corner to the center

File: urdf/marmotte.urdf.xacro (robot description, xacro)
@@ -3,5 +3,5 @@
   <xacro:property name="M_PI" value="3.14159"/>
   <!-- horizontal, horizontal_90, vertical -->
-  <xacro:property name="configuration" value="horizontal"/>
+  <xacro:property name="configuration" value="horizontal_90"/>
   <link name="base_link"/>
   <xacro:if value="${configuration != 'vertical'}">
@@ -25,8 +25,8 @@
   <joint name="lidar_imu_board_joint" type="fixed">
       <xacro:if value="${configuration != 'horizontal_90'}">
-        <origin xyz="0 0 0.039" rpy="0 0 0" />
+        <origin xyz="0.06 -0.06 0.039" rpy="0 0 0" />
       </xacro:if>
       <xacro:if value="${configuration == 'horizontal_90'}">
-        <origin xyz="0 0 0.039" rpy="0 0 ${M_PI/2}" />
+        <origin xyz="0.06 -0.06 0.039" rpy="0 0 ${M_PI/2}" />
       </xacro:if>
       <xacro:if value="${configuration != 'vertical'}">
@@ -40,5 +40,5 @@
   <link name="lslidarc16"/>
   <joint name="lslidarc16_joint" type="fixed">
-    <origin xyz="0.06 -0.06 0.036" rpy="0 0 ${M_PI/2}" />
+    <origin xyz="0 0 0.036" rpy="0 0 ${M_PI}" />
     <parent link="lidar_imu_board" />
     <child link="lslidarc16" />
@@ -46,5 +46,5 @@
   <link name="imu"/>
   <joint name="imu_joint" type="fixed">
-    <origin xyz="0.039254 -0.04274357 -0.0161" rpy="${M_PI} 0 0" />
+    <origin xyz="-0.02075 0.01726 -0.0161" rpy="${M_PI} 0 0" />
     <parent link="lidar_imu_board" />
     <child link="imu" />

Commit message: Edit values for vertical mount

File: urdf/marmotte.urdf.xacro (robot description, xacro)
@@ -17,5 +17,5 @@
     <link name="lidar_imu_mount_vertical"/>
     <joint name="lidar_imu_mount_vertical_joint" type="fixed">
-        <origin xyz="0.17834 -0.02 0.38378" rpy="${M_PI/2} 0.178 0" />
+        <origin xyz="0.17883 -0.02 0.36878" rpy="${M_PI/2} 0.178 0" />
         <parent link="base_link" />
         <child link="lidar_imu_mount_vertical" />

Commit message: Edit values for verical mount

File: urdf/marmotte.urdf.xacro (robot description, xacro)
@@ -17,5 +17,5 @@
     <link name="lidar_imu_mount_vertical"/>
     <joint name="lidar_imu_mount_vertical_joint" type="fixed">
-        <origin xyz="0.17883 -0.02 0.36878" rpy="${M_PI/2} 0.178 0" />
+        <origin xyz="0.17883 -0.02 0.36878" rpy="${M_PI/2} 0 0" />
         <parent link="base_link" />
         <child link="lidar_imu_mount_vertical" />

Commit message: Change IMU's link name to mti100

File: urdf/marmotte.urdf.xacro (robot description, xacro)
@@ -3,5 +3,5 @@
   <xacro:property name="M_PI" value="3.14159"/>
   <!-- horizontal, horizontal_90, vertical -->
-  <xacro:property name="configuration" value="horizontal_90"/>
+  <xacro:property name="configuration" value="horizontal"/>
   <link name="base_link"/>
   <xacro:if value="${configuration != 'vertical'}">
@@ -44,9 +44,9 @@
     <child link="lslidarc16" />
   </joint>
-  <link name="imu"/>
+  <link name="mti100"/>
   <joint name="imu_joint" type="fixed">
     <origin xyz="-0.02075 0.01726 -0.0161" rpy="${M_PI} 0 0" />
     <parent link="lidar_imu_board" />
-    <child link="imu" />
+    <child link="mti100" />
   </joint>
   <link name="realsense_link"/>

Commit message: Replace lslidar with velodyne

File: urdf/marmotte.urdf.xacro (robot description, xacro)
@@ -38,9 +38,9 @@
       <child link="lidar_imu_board" />
   </joint>
-  <link name="lslidarc16"/>
-  <joint name="lslidarc16_joint" type="fixed">
-    <origin xyz="0 0 0.036" rpy="0 0 ${M_PI}" />
+  <link name="velodyne"/>
+  <joint name="velodyne_joint" type="fixed">
+    <origin xyz="0 0 0.0377" rpy="0 0 ${-M_PI/2}" />
     <parent link="lidar_imu_board" />
-    <child link="lslidarc16" />
+    <child link="velodyne" />
   </joint>
   <link name="mti100"/>

Commit message: Fix yaw angle from datasheet

File: urdf/marmotte.urdf.xacro (robot description, xacro)
@@ -40,5 +40,6 @@
   <link name="velodyne"/>
   <joint name="velodyne_joint" type="fixed">
-    <origin xyz="0 0 0.0377" rpy="0 0 ${-M_PI/2}" />
+    <!-- <origin xyz="0 0 0.0377" rpy="0 0 ${-M_PI/2}" /> -->
+    <origin xyz="0 0 0.0377" rpy="0 0 0" />
     <parent link="lidar_imu_board" />
     <child link="velodyne" />

Commit message: fix orientation of velodyne lidar

File: urdf/marmotte.urdf.xacro (robot description, xacro)
@@ -40,5 +40,4 @@
   <link name="velodyne"/>
   <joint name="velodyne_joint" type="fixed">
-    <!-- <origin xyz="0 0 0.0377" rpy="0 0 ${-M_PI/2}" /> -->
     <origin xyz="0 0 0.0377" rpy="0 0 0" />
     <parent link="lidar_imu_board" />

Commit message: Pushed modifications on marmotte before ROS2

File: urdf/marmotte.urdf.xacro (robot description, xacro)
@@ -1,61 +1,172 @@
-<?xml version="1.0"?>
+<?xml version="1.0" ?>
 <robot name="marmotte" xmlns:xacro="http://ros.org/wiki/xacro">
-  <xacro:property name="M_PI" value="3.14159"/>
-  <!-- horizontal, horizontal_90, vertical -->
-  <xacro:property name="configuration" value="horizontal"/>
+  <xacro:include filename="$(find kinova_description)/urdf/j2n6s300.xacro"/>
+  <xacro:include filename="$(find marmotte_description)/urdf/sensors.urdf.xacro"/>
+  <xacro:include filename="$(find realsense2_description)/urdf/_d435i.urdf.xacro"/>
+  <!-- JACO j2n6s300 -->
+  <xacro:j2n6s300  base_parent="base_arm"/>
+  <!-- REALSENSE ARM -->
+  <xacro:property name="realsense_angle_rad" value="${M_PI/6}" />
+  <xacro:sensor_d435i parent="j2n6s300_link_6" name="realsense" use_nominal_extrinsics="false">
+    <origin xyz="0.1095 0 -0.0381" rpy="0 ${M_PI/2+realsense_angle_rad} 0"/>
+  </xacro:sensor_d435i>
+  <joint name="base_link_intial_joint" type="fixed">
+    <parent link="base_link"/>
+    <child link="base_link_chassis_CAD"/>
+    <origin xyz="0 0  0" rpy="0 0 0"/>
+  </joint>
+  <joint name="base_link_to_sensor_rack" type="fixed">
+    <parent link="base_link_chassis_CAD"/>
+    <child link="sensor_rack_CAD"/>
+    <origin xyz="-0.19853 -0.19824  0.06899" rpy="0.e+00  0.e+00 -1.e-05"/>
+    <axis xyz="0 0 0"/>
+    <limit lower="0" upper="0" effort="0" velocity="0"/>
+  </joint>
+  <joint name="left_track_j" type="fixed">
+    <parent link="base_link_chassis_CAD"/>
+    <child link="left_track_CAD"/>
+    <origin xyz="0   0.26 0" rpy="0 0 0"/>
+    <axis xyz="0 0 0"/>
+    <limit lower="0" upper="0" effort="0" velocity="0"/>
+  </joint>
+  <joint name="right_track_j" type="fixed">
+    <parent link="base_link_chassis_CAD"/>
+    <child link="right_track_CAD"/>
+    <origin xyz="0   -0.26  0" rpy="0 0 0"/>
+    <axis xyz="0 0 0"/>
+    <limit lower="0" upper="0" effort="0" velocity="0"/>
+  </joint>
+  <!-- JOINT BETWEEN ARM AND BODY -->
+  <joint name="body_arm" type="fixed">
+    <parent link="base_link"/>
+    <child link="base_arm"/>
+    <origin xyz="-0.072 0.02 0.326" rpy="0 0 ${M_PI}"/>
+    <axis xyz="0 0 0"/>
+  </joint>
+  <!---->
+  <joint name="base_basket" type="fixed">
+    <parent link="base_link"/>
+    <child link="basket_visualize"/>
+    <origin xyz="-0.2765 0 0.1" rpy="0 0 0"/>
+  </joint>
+  <link name="base_arm"/>
   <link name="base_link"/>
-  <xacro:if value="${configuration != 'vertical'}">
-    <link name="lidar_imu_mount_horizontal"/>
-    <joint name="lidar_imu_mount_horizontal_joint" type="fixed">
-        <origin xyz="0.19834 0.06 0.26011" rpy="0 0.178 0" />
-        <parent link="base_link" />
-        <child link="lidar_imu_mount_horizontal" />
-    </joint>
-  </xacro:if>
-  <!-- Vertical board -->
-  <xacro:if value="${configuration == 'vertical'}">
-    <link name="lidar_imu_mount_vertical"/>
-    <joint name="lidar_imu_mount_vertical_joint" type="fixed">
-        <origin xyz="0.17883 -0.02 0.36878" rpy="${M_PI/2} 0 0" />
-        <parent link="base_link" />
-        <child link="lidar_imu_mount_vertical" />
-    </joint>
-  </xacro:if>
-  <link name="lidar_imu_board"/>
-  <joint name="lidar_imu_board_joint" type="fixed">
-      <xacro:if value="${configuration != 'horizontal_90'}">
-        <origin xyz="0.06 -0.06 0.039" rpy="0 0 0" />
-      </xacro:if>
-      <xacro:if value="${configuration == 'horizontal_90'}">
-        <origin xyz="0.06 -0.06 0.039" rpy="0 0 ${M_PI/2}" />
-      </xacro:if>
-      <xacro:if value="${configuration != 'vertical'}">
-        <parent link="lidar_imu_mount_horizontal" />
-      </xacro:if>
-      <xacro:if value="${configuration == 'vertical'}">
-        <parent link="lidar_imu_mount_vertical" />
-      </xacro:if>
-      <child link="lidar_imu_board" />
-  </joint>
-  <link name="velodyne"/>
-  <joint name="velodyne_joint" type="fixed">
-    <!-- <origin xyz="0 0 0.0377" rpy="0 0 ${-M_PI/2}" /> -->
-    <origin xyz="0 0 0.0377" rpy="0 0 0" />
-    <parent link="lidar_imu_board" />
-    <child link="velodyne" />
-  </joint>
-  <link name="mti100"/>
-  <joint name="imu_joint" type="fixed">
-    <origin xyz="-0.02075 0.01726 -0.0161" rpy="${M_PI} 0 0" />
-    <parent link="lidar_imu_board" />
-    <child link="mti100" />
-  </joint>
-  <link name="realsense_link"/>
-  <joint name="realsense_joint" type="fixed">
-    <origin xyz="-0.31593 -0.0175 0.34488" rpy="0 0.558505 ${M_PI}" />
-    <parent link="base_link" />
-    <child link="realsense_link" />
-  </joint>
-  <!-- Cameras -->
-  <xacro:include filename="$(find marmotte_description)/urdf/cameras.urdf.xacro"/>
+  <material name="black">
+    <color rgba="0.0 0.0 0.0 1.0"/>
+  </material>
+  <link name="basket_visualize">
+    <collision name="basket_visualize_collision">
+      <origin xyz="0    0    0" rpy="0 0 0"/>
+      <geometry>
+        <box size="0.193 0.393 0.02"/>
+      </geometry>
+    </collision>
+    <visual name="basket_visualize_visual">
+      <origin xyz="0     0    0" rpy="0   0   0"/>
+      <geometry>
+        <box size="0.193 0.393 0.02"/>
+      </geometry>
+      <material name="black"/>
+    </visual>
+  </link>
+  <link name="base_link_chassis_CAD">
+    <inertial>
+      <mass value="29.053"/>
+      <origin xyz="0 0 0" rpy="0 0 0"/>
+      <inertia ixx="2.411" ixy="0.0" ixz="0.0" iyy="4.173" iyz="0.0" izz="4.745"/>
+    </inertial>
+    <collision name="base_link_collision_bottom">
+      <origin xyz="0    0    0.046" rpy="0 0 0"/>
+      <geometry>
+        <box size="0.80 0.5709 0.2"/>
+      </geometry>
+    </collision>
+    <visual name="Body_visual">
+      <origin xyz="0     0    -0.135" rpy="0   0   1.57"/>
+      <geometry>
+        <mesh filename="package://marmotte_description/meshes/hd2_marble_base_body_metric.dae" scale="1.0 1.0 1.0"/>
+      </geometry>
+    </visual>
+  </link>
+  <link name="sensor_rack_CAD">
+    <inertial>
+      <mass value="10.40255"/>
+      <origin xyz="0.28 0.2  0.06" rpy="0 0 0"/>
+      <inertia ixx="0.193" ixy="-0.0031" ixz="0.00912" iyy="0.301" iyz="0.00313" izz="0.35676"/>
+    </inertial>
+    <collision name="collision_base">
+      <origin xyz="0.275 0.2   0.075" rpy="0 0 0"/>
+      <geometry>
+        <box size="0.56 0.4 0.15"/>
+      </geometry>
+    </collision>
+    <collision name="collision_top">
+      <origin xyz="0.15  0.2   0.215" rpy="0 0 0"/>
+      <geometry>
+        <box size="0.28 0.4 0.13"/>
+      </geometry>
+    </collision>
+    <collision name="collision_laser">
+      <origin xyz="0.505 0.2   0.17" rpy="0   0.17 0"/>
+      <geometry>
+        <box size="0.135 0.13 0.13"/>
+      </geometry>
+    </collision>
+    <visual name="visual">
+      <origin xyz="0 0 0" rpy="0 0 0"/>
+      <geometry>
+        <mesh filename="package://marmotte_description/meshes/sensor_rack_lowres_shallow_laser.dae" scale="1 1 1"/>
+      </geometry>
+    </visual>
+  </link>
+  <link name="left_track_CAD">
+    <inertial>
+      <mass value="6.0"/>
+      <origin xyz="0 0 0" rpy="0 0 0"/>
+      <inertia ixx="0.03828" ixy="0" ixz="0" iyy="0.2925" iyz="0" izz="0.2642"/>
+    </inertial>
+    <collision name="front_left_wheel_link_collision">
+      <origin xyz="0.36 0   0" rpy="1.57079 0      0"/>
+      <geometry>
+        <cylinder radius="0.129" length="0.1"/>
+      </geometry>
+    </collision>
+    <collision name="rear_left_wheel_link_collision">
+      <origin xyz="-0.36  0    0" rpy="1.57079 0      0"/>
+      <geometry>
+        <cylinder radius="0.129" length="0.1"/>
+      </geometry>
+    </collision>
+    <collision name="left_track_box_collision">
+      <origin xyz="0 0 0" rpy="0 0 0"/>
+      <geometry>
+        <box size="0.72 0.1 0.258"/>
+      </geometry>
+    </collision>
+  </link>
+  <link name="right_track_CAD">
+    <inertial>
+      <mass value="6.0"/>
+      <origin xyz="0 0 0" rpy="0 0 0"/>
+      <inertia ixx="0.03828" ixy="0" ixz="0" iyy="0.2925" iyz="0" izz="0.2642"/>
+    </inertial>
+    <collision name="front_right_wheel_link_collision">
+      <origin xyz="0.36 0   0" rpy="1.57079 0      0"/>
+      <geometry>
+        <cylinder radius="0.129" length="0.1"/>
+      </geometry>
+    </collision>
+    <collision name="rear_right_wheel_link_collision">
+      <origin xyz="-0.36  0    0" rpy="1.57079 0      0"/>
+      <geometry>
+        <cylinder radius="0.129" length="0.1"/>
+      </geometry>
+    </collision>
+    <collision name="right_track_box_collision">
+      <origin xyz="0 0 0" rpy="0 0 0"/>
+      <geometry>
+        <box size="0.72 0.1 0.258"/>
+      </geometry>
+    </collision>
+  </link>
 </robot>
