Commit message: Renamed IMU joints and links to match IMU messages

File: urdf/sensors.urdf.xacro (robot description, xacro)
@@ -48,5 +48,5 @@
          <origin xyz="-0.02075 0.01726 -0.0161" rpy="${M_PI} 0 0" />
          <parent link="lidar_imu_board" />
-         <child link="mti100" />
+         <child link="imu" />
       </joint>
    <link name="lidar_imu_board"/>
@@ -58,12 +58,12 @@
          <child link="lidar_link" />
       </joint>
-      <joint name="mti100_joint" type="fixed">
+      <joint name="imu_joint" type="fixed">
          <origin xyz="-0.05718 -0.103 0.2885" rpy="0 0 0" />
          <parent link="base_link" />
-         <child link="mti100" />
+         <child link="imu" />
       </joint>
    </xacro:unless>
    <link name="lidar_link"/>
-   <link name="mti100"/>
+   <link name="imu"/>
    <link name="camera0_link"/>
    <link name="camera1_link"/>

Commit message: Fix IMU and lidar tfs

File: urdf/sensors.urdf.xacro (robot description, xacro)
@@ -3,5 +3,5 @@
    <xacro:property name="M_PI" value="3.1415926535897931"/>
    <xacro:property name="length_cam" value="0.05" />
-   <xacro:property name="configuration_horizon_or_vert" value="false"/>      <!-- True: horiz or vert/ False: old without imu  -->
+   <xacro:property name="configuration_horizon_or_vert" value="true"/>      <!-- True: horiz or vert/ False: old without imu  -->
    <xacro:property name="configuration" value="horizontal"/>      <!-- horizontal, horizontal_90, vertical -->
    <xacro:if value="${configuration_horizon_or_vert}">
@@ -40,6 +40,5 @@
       </joint>
       <joint name="lidar_link_joint" type="fixed">
-         <!-- <origin xyz="0 0 0.0377" rpy="0 0 ${-M_PI/2}" /> -->
-         <origin xyz="0 0 0.0377" rpy="0 0 0" />
+          <origin xyz="0 0 0.0377" rpy="0 0 ${M_PI}" />
          <parent link="lidar_imu_board" />
          <child link="lidar_link" />

Commit message: Update pitch value with Vachon loop calibration result

File: urdf/sensors.urdf.xacro (robot description, xacro)
@@ -45,5 +45,5 @@
       </joint>
       <joint name="imu_joint" type="fixed">
-         <origin xyz="-0.02075 0.01726 -0.0161" rpy="${M_PI} 0 0" />
+         <origin xyz="-0.02075 0.01726 -0.0161" rpy="${M_PI} 0.022837797 0" /> <!-- Calibration done on March 16th loop around vachon rosbag: rosbag2_2023_03_16-13_24_06 -->
          <parent link="lidar_imu_board" />
          <child link="imu" />

Commit message: Fix IMU calibration with new changes

File: urdf/sensors.urdf.xacro (robot description, xacro)
@@ -10,5 +10,5 @@
          <link name="lidar_imu_mount_horizontal"/>
          <joint name="lidar_imu_mount_horizontal_joint" type="fixed">
-            <origin xyz="0.19834 0.06 0.26011" rpy="0 0.178 0" />
+            <origin xyz="0.19834 0.06 0.26011" rpy="0 0.174533 0" />
             <parent link="base_link" />
             <child link="lidar_imu_mount_horizontal" />
@@ -45,5 +45,5 @@
       </joint>
       <joint name="imu_joint" type="fixed">
-         <origin xyz="-0.02075 0.01726 -0.0161" rpy="${M_PI} 0.022837797 0" /> <!-- Calibration done on March 16th loop around vachon rosbag: rosbag2_2023_03_16-13_24_06 -->
+         <origin xyz="-0.02075 0.01726 -0.0161" rpy="${M_PI} 0.031454056 0" />
          <parent link="lidar_imu_board" />
          <child link="imu" />

Commit message: Freeze marmotte git repos for SNOW demo

File: urdf/sensors.urdf.xacro (robot description, xacro)
@@ -45,5 +45,5 @@
       </joint>
       <joint name="imu_joint" type="fixed">
-         <origin xyz="-0.02075 0.01726 -0.0161" rpy="${M_PI} 0.031454056 0" />
+         <origin xyz="-0.02075 0.01726 -0.0161" rpy="${M_PI} 0 0" />
          <parent link="lidar_imu_board" />
          <child link="imu" />

Commit message: Added barometric pressure dps sensor to the urdf

File: urdf/sensors.urdf.xacro (robot description, xacro)
@@ -118,3 +118,9 @@
       <child link="realsense_link" />
   </joint> -->
+  <link name="dps310_marmotte" />
+  <joint name="dps310_marmotte_joint" type="fixed">
+    <origin xyz="0.335 0.02 0.02" rpy="0 0.174533 0" />
+    <parent link="lidar_link" />
+    <child link="dps310_marmotte" />
+  </joint>
 </robot>
