Commit message: modified some stuff in the urdf to fit what we changed on marmotte.

File: urdf/sensors_new.urdf.xacro (robot description, xacro)
@@ -12,5 +12,5 @@
             <!-- <origin xyz="-0.19466 0.06 0.41811" rpy="0 0.174533 ${M_PI}" /> -->
             <!-- <origin xyz="0.19834 0.06 0.26011" rpy="0 0.174533 0" /> -->
-            <origin xyz="0.19834 0.06 0.346975" rpy="0 0 0" />
+            <origin xyz="-0.08866 0 0.393975" rpy="0 0 ${M_PI}" />
             <parent link="base_link" />
             <child link="lidar_imu_mount_horizontal" />
@@ -123,5 +123,5 @@
   <link name="dps310_marmotte" />
   <joint name="dps310_marmotte_joint" type="fixed">
-    <origin xyz="0.305 -0.02 -0.085" rpy="0 0.0 0" />
+    <origin xyz="-0.115 -0.02 -0.122" rpy="0 0.0 0" />
     <parent link="lidar_link" />
     <child link="dps310_marmotte" />

Commit message: corrected imu orientation

File: urdf/sensors_new.urdf.xacro (robot description, xacro)
@@ -47,5 +47,5 @@
       </joint>
       <joint name="imu_joint" type="fixed">
-         <origin xyz="-0.02075 0.01726 -0.0161" rpy="${M_PI} 0.0 0" />
+         <origin xyz="-0.02075 0.01726 -0.0161" rpy="${M_PI} 0.0 ${M_PI}" />
          <!-- <origin xyz="-0.02075 0.01726 -0.0161" rpy="${M_PI} 0.031454056 0" /> -->
          <parent link="lidar_imu_board" />
